File: Electronics/SmootherBoard/SmootherBoard.kicad_pcb (KiCad board)
At the start: 2 copper layers, 58 parts, among them SW1 SW_Push, SW2 SW_Push, U1 ESP32-DEVKITC-32D, U10 CNY70, U11 CNY70, U12 CNY70, U13 CNY70, U14 AP7363-33, U2 MPU6050_breakdown, U3 CNY70, U4 TP4056_module, U5 CNY70, U6 CNY70, U7 DRV8833_module, U8 DRV8833_module, U9 CNY70

Commit message: Board first completed.
Parts:
- C1, C2, C3, C4, C5, G***, L1, R1, R10, R11, R12, R13, R14, R15, R16, R17, R18, R19, R2, R20, R21, R22, R23, R25, R26, R28, R4, R5, R6, R8, R9, U10, U11, U12, U13, U14, U3, U5, U6, U9: moved to B.Cu
- moved Motor2 158.3 mm to (186.7, 141.0), turned to 180 degrees
- moved R20 156.4 mm to (210.6, 125.7)
- moved R18 148.8 mm to (210.6, 120.7)
- moved G*** 132.2 mm to (203.2, 111.8), turned to 270 degrees
- moved R21 131.0 mm to (181.6, 60.7), turned to 90 degrees
- moved C5 130.7 mm to (189.2, 86.1), turned to 270 degrees
- moved R19 130.4 mm to (210.6, 123.2)
- moved R25 127.2 mm to (191.8, 60.7), turned to 90 degrees
- moved R27 125.8 mm to (191.8, 60.7), turned to 90 degrees
- moved C6 123.9 mm to (185.4, 85.4), turned to 270 degrees
- moved R13 123.5 mm to (185.4, 133.1), turned to 90 degrees
- moved R9 122.8 mm to (210.6, 118.1)
- moved U6 122.1 mm to (179.1, 137.2)
- moved R23 120.7 mm to (183.9, 66.0)
- moved BT1 119.4 mm to (201.9, 74.0), turned to 270 degrees
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Other:
- board outline added: 63.5 x 94 mm
- board text added: "Smoother V1.0"

Commit message: Generated manufacturing files.
Parts:
- added J1: Conn_01x02_Male, Connector_PinHeader_2.54mm:PinHeader_1x02_P2.54mm_Vertical, F.Cu at (214.6, 87.6)
Connections:
- U4 pad 6: BatV -> Net-(J1-Pad2)
Routing:
- net GND: track 0.00 -> 309.8 mm, vias 0 -> 25
- net +3V3: track 0.00 -> 220.1 mm
- net BatV: track 0.00 -> 115.9 mm, vias 0 -> 1
- net Motor0A: track 0.00 -> 93.8 mm
- net Net-(Motor0-Pad2): track 0.00 -> 91.8 mm, vias 0 -> 1
- net Motor0B: track 0.00 -> 82.0 mm, vias 0 -> 1
- net LineSensor0: track 0.00 -> 80.6 mm, vias 0 -> 1
- net SW0: track 0.00 -> 79.9 mm
- net LineSensor1: track 0.00 -> 79.9 mm, vias 0 -> 1
- net Net-(Motor2-Pad1): track 0.00 -> 76.2 mm
- net WheelEnc1: track 0.00 -> 72.5 mm, vias 0 -> 1
- net LineSensor2: track 0.00 -> 68.4 mm, vias 0 -> 1
- net SW1: track 0.00 -> 66.2 mm
- net Net-(BT1-Pad2): track 0.00 -> 63.9 mm
- net Motor1A: track 0.00 -> 62.5 mm, vias 0 -> 1
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- added copper zone on B.Cu, net GND
- added copper zone on F.Cu, net GND

Commit message: Changed LDO package for sot-252.
Parts:
- U14: footprint Package_TO_SOT_SMD:SOT-223-3_TabPin2 -> Package_TO_SOT_SMD:TO-252-3_TabPin2
- moved U14 1.86 mm to (205.7, 90.2)
Routing:
- net Net-(Motor2-Pad2): track 52.7 -> 111.9 mm
- net GND: track 309.8 -> 358.1 mm, vias 25 -> 23
- net +3V3: track 220.1 -> 267.5 mm, vias 0 -> 1
- net MotorSleep: track 51.9 -> 35.7 mm
- net Net-(J1-Pad2): track 50.3 -> 65.8 mm
- net WheelEnc1: track 72.5 -> 86.6 mm
- net Motor0A: track 93.8 -> 83.4 mm, vias 0 -> 2
- net Motor3B: track 27.0 -> 36.9 mm, vias 0 -> 1
- net Net-(Motor0-Pad2): track 91.8 -> 99.4 mm, vias 1 -> 3
- net BatV: track 115.9 -> 108.4 mm, vias 1 -> 2
- net LineSensor0: track 80.6 -> 87.6 mm
- net Net-(Motor2-Pad1): track 76.2 -> 70.4 mm
- net BAT-Sense: track 33.6 -> 28.1 mm
- net SDA: track 35.6 -> 30.3 mm
- net MPU_inter: track 54.8 -> 49.5 mm, vias 0 -> 1
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- added copper zone on B.Cu, net (none)
- removed copper zone on B.Cu, net GND
Other:
- net class Power added: clearance 0.2, trace_width 1, via_dia 1.6, via_drill 0.8
